Commit message: homologation with task list adjusted

File: src/holonomic_robot_description/urdf/holonomic_robot.urdf (robot description, URDF)
Before this commit: robot holonomic_robot, 6 links, 5 joints
Joints:
- joint lidar_joint: origin xyz=0 0 0.075 rpy=0 0 0 -> xyz=0 0 0.075 rpy=0 0 3.14159

Commit message: nav2 params

File: src/holonomic_robot_description/urdf/holonomic_robot.urdf (robot description, URDF)
Before this commit: robot holonomic_robot, 6 links, 5 joints
Joints:
- joint lidar_joint: origin xyz=0 0 0.075 rpy=0 0 3.14159 -> xyz=0 0 0 rpy=0 0 3.14
